File: Production/Qwiic 1x1/SparkFun_Pressure_Sensor_BMP581_Qwiic-Panel.brd (EAGLE design)
At the start: 175 x 117.3 mm, 1134 parts, among them J1 QWIIC_RIGHT_ANGLE, J10 QWIIC_RIGHT_ANGLE, J11 QWIIC_RIGHT_ANGLE, J13 QWIIC_RIGHT_ANGLE, J14 QWIIC_RIGHT_ANGLE, J16 QWIIC_RIGHT_ANGLE, J17 QWIIC_RIGHT_ANGLE, J19 QWIIC_RIGHT_ANGLE, J2 QWIIC_RIGHT_ANGLE, J20 QWIIC_RIGHT_ANGLE, J22 QWIIC_RIGHT_ANGLE, J23 QWIIC_RIGHT_ANGLE, J25 QWIIC_RIGHT_ANGLE, J26 QWIIC_RIGHT_ANGLE, J28 QWIIC_RIGHT_ANGLE, J29 QWIIC_RIGHT_ANGLE, J31 QWIIC_RIGHT_ANGLE, J32 QWIIC_RIGHT_ANGLE, J34 QWIIC_RIGHT_ANGLE, J35 QWIIC_RIGHT_ANGLE, J37 QWIIC_RIGHT_ANGLE, J38 QWIIC_RIGHT_ANGLE, J4 QWIIC_RIGHT_ANGLE, J40 QWIIC_RIGHT_ANGLE, J41 QWIIC_RIGHT_ANGLE, J43 QWIIC_RIGHT_ANGLE, J44 QWIIC_RIGHT_ANGLE, J46 QWIIC_RIGHT_ANGLE, J47 QWIIC_RIGHT_ANGLE, J49 QWIIC_RIGHT_ANGLE, J5 QWIIC_RIGHT_ANGLE, J50 QWIIC_RIGHT_ANGLE, J52 QWIIC_RIGHT_ANGLE, J53 QWIIC_RIGHT_ANGLE, J55 QWIIC_RIGHT_ANGLE, J56 QWIIC_RIGHT_ANGLE, J58 QWIIC_RIGHT_ANGLE, J59 QWIIC_RIGHT_ANGLE, J61 QWIIC_RIGHT_ANGLE, J62 QWIIC_RIGHT_ANGLE, J64 QWIIC_RIGHT_ANGLE, J65 QWIIC_RIGHT_ANGLE, J67 QWIIC_RIGHT_ANGLE, J68 QWIIC_RIGHT_ANGLE, J7 QWIIC_RIGHT_ANGLE, J70 QWIIC_RIGHT_ANGLE, J71 QWIIC_RIGHT_ANGLE, J8 QWIIC_RIGHT_ANGLE, U1 BMP581, U10 BMP581, U11 BMP581, U12 BMP581, U13 BMP581, U14 BMP581, U15 BMP581, U16 BMP581, U17 BMP581, U18 BMP581, U19 BMP581, U2 BMP581, U20 BMP581, U21 BMP581, U22 BMP581, U23 BMP581, U24 BMP581, U3 BMP581, U4 BMP581, U5 BMP581, U6 BMP581, U7 BMP581, U8 BMP581, U9 BMP581

Commit message: Add production files for reds
Parts:
- added JP73, JP77, JP81, JP85, JP89, JP93: ADR, SparkFun-Jumpers:SMT-JUMPER_3_1-NC_TRACE_SILK
- added JP74, JP78, JP82, JP86, JP90, JP94: I2C, SparkFun-Jumpers:SMT-JUMPER_3_2-NC_TRACE_SILK
- added JP75, JP79, JP83, JP87, JP91, JP95: LED, SparkFun-Jumpers:SMT-JUMPER_2_NC_TRACE_SILK
- added JP76, JP80, JP84, JP88, JP92, JP96: !CSB!, SparkFun-Jumpers:SMT-JUMPER_2_NC_TRACE_SILK
- added R121, R122, R127, R128, R133, R134, R139, R140: 2.2k, SparkFun-Resistors:0603
- added R123, R124, R126, R129, R130, R132, R135, R136, R138, R141, R142, R144: 10k, SparkFun-Resistors:0603
- added R125, R131, R137, R143: 1k, SparkFun-Resistors:0603
- added U$553, U$575, U$578, U$600: (no value), output:BMP5810
- added U$554, U$555, U$579, U$580: (no value), output:#GND#0
- added U$556, U$557, U$581, U$582: (no value), output:#SDI#SDA#0
- added U$558, U$559, U$583, U$584: (no value), output:#SCK#SCL#0
- added U$560, U$561, U$585, U$586: (no value), output:#SDO#ADR#0
- added U$562, U$563, U$587, U$588: (no value), output:#INT#0
- added U$564, U$565, U$589, U$590: (no value), output:#3V3#0
- added U$566, U$567, U$591, U$592: (no value), output:##CSB##0
- added U$568, U$593: (no value), output:#ADR#0
- added U$569, U$594: (no value), output:#LED#0
- added U$570, U$595: (no value), output:#I2C#0
- added U$571, U$596: (no value), output:#0X46#0
- added U$572, U$597: (no value), output:#0X47#0
- added U$573, U$598: (no value), output:PWR0
- added U$574, U$599: (no value), output:##CSB##1
- added U$576: (no value), output:PRESSURE0
- added U$577: (no value), output:SENSOR0
- JP10, JP22, JP34, JP46, JP58, JP70: value ADR -> I2C; device SparkFun-Jumpers:SMT-JUMPER_3_1-NC_TRACE_SILK -> SparkFun-Jumpers:SMT-JUMPER_3_2-NC_TRACE_SILK
- JP11, JP23, JP35, JP47, JP59, JP71: value I2C -> LED; device SparkFun-Jumpers:SMT-JUMPER_3_2-NC_TRACE_SILK -> SparkFun-Jumpers:SMT-JUMPER_2_NC_TRACE_SILK
- JP12, JP24, JP36, JP48, JP60, JP72: value LED -> !CSB!
- JP16, JP28, JP4, JP40, JP52, JP64: value ADR -> !CSB!; device SparkFun-Jumpers:SMT-JUMPER_3_1-NC_TRACE_SILK -> SparkFun-Jumpers:SMT-JUMPER_2_NC_TRACE_SILK
- JP17, JP29, JP41, JP5, JP53, JP65: value I2C -> ADR; device SparkFun-Jumpers:SMT-JUMPER_3_2-NC_TRACE_SILK -> SparkFun-Jumpers:SMT-JUMPER_3_1-NC_TRACE_SILK
- JP18, JP30, JP42, JP54, JP6, JP66: value LED -> I2C; device SparkFun-Jumpers:SMT-JUMPER_2_NC_TRACE_SILK -> SparkFun-Jumpers:SMT-JUMPER_3_2-NC_TRACE_SILK
- JP19, JP31, JP43, JP55, JP67, JP7: value ADR -> LED; device SparkFun-Jumpers:SMT-JUMPER_3_1-NC_TRACE_SILK -> SparkFun-Jumpers:SMT-JUMPER_2_NC_TRACE_SILK
- JP20, JP32, JP44, JP56, JP68, JP8: value I2C -> !CSB!; device SparkFun-Jumpers:SMT-JUMPER_3_2-NC_TRACE_SILK -> SparkFun-Jumpers:SMT-JUMPER_2_NC_TRACE_SILK
- JP21, JP33, JP45, JP57, JP69, JP9: value LED -> ADR; device SparkFun-Jumpers:SMT-JUMPER_2_NC_TRACE_SILK -> SparkFun-Jumpers:SMT-JUMPER_3_1-NC_TRACE_SILK
- R10, R100, R105, R120, R15, R30, R40, R45, R60, R70, R75, R90: value 1k -> 10k
- R101, R107, R11, R17, R41, R47, R71, R77: value 2.2k -> 1k
- R102, R106, R111, R112, R117, R12, R16, R21, R22, R27, R36, R42, R46, R51, R52, R57, R6, R66, R72, R76, R81, R82, R87, R96: value 2.2k -> 10k
- R103, R104, R109, R13, R14, R19, R38, R43, R44, R49, R68, R73, R74, R79, R8, R98: value 10k -> 2.2k
- R110, R115, R20, R25, R50, R55, R80, R85: value 1k -> 2.2k
- R113, R119, R23, R29, R53, R59, R83, R89: value 10k -> 1k
- U$100, U$353, U$400, U$78: device output:#SCK#SCL#0 -> output:BMP5810
- U$101, U$376: device output:#SCK#SCL#0 -> output:PRESSURE0
- U$102, U$402: device output:#SDO#ADR#0 -> output:SENSOR0
- U$103, U$125, U$378, U$425: device output:#SDO#ADR#0 -> output:BMP5810
- U$104, U$105, U$380, U$404: device output:#INT#0 -> output:#GND#0
- U$106, U$107, U$382, U$406: device output:#3V3#0 -> output:#SDI#SDA#0
- U$108, U$109, U$384, U$408: device output:##CSB##0 -> output:#SCK#SCL#0
- U$110, U$386: device output:#ADR#0 -> output:#SDO#ADR#0
- U$111, U$410: device output:#LED#0 -> output:#SDO#ADR#0
- U$112, U$388: device output:#I2C#0 -> output:#INT#0
- U$113, U$412: device output:#0X46#0 -> output:#INT#0
- U$114, U$390: device output:#0X47#0 -> output:#3V3#0
- U$115, U$414: device output:PWR0 -> output:#3V3#0
- U$116, U$392: device output:PRESSURE0 -> output:##CSB##0
- U$117, U$416: device output:SENSOR0 -> output:##CSB##0
- U$118: device output:BMP5810 -> output:#ADR#0
- U$119, U$419: device output:#GND#0 -> output:#LED#0
- U$120, U$395: device output:#GND#0 -> output:#I2C#0
- U$121, U$421: device output:#SDI#SDA#0 -> output:#0X46#0
- U$122, U$397: device output:#SDI#SDA#0 -> output:#0X47#0
- U$123, U$423: device output:#SCK#SCL#0 -> output:PWR0
- U$124, U$399: device output:#SCK#SCL#0 -> output:##CSB##1
- U$126, U$401: device output:#SDO#ADR#0 -> output:PRESSURE0
- U$127, U$427: device output:#INT#0 -> output:SENSOR0
- U$128, U$150, U$403, U$450: device output:#INT#0 -> output:BMP5810
- U$129, U$130, U$405, U$429: device output:#3V3#0 -> output:#GND#0
- U$131, U$132, U$407, U$431: device output:##CSB##0 -> output:#SDI#SDA#0
- U$133, U$409: device output:#ADR#0 -> output:#SCK#SCL#0
- U$134, U$433: device output:#LED#0 -> output:#SCK#SCL#0
- U$135, U$411: device output:#I2C#0 -> output:#SDO#ADR#0
- U$136, U$435: device output:#0X46#0 -> output:#SDO#ADR#0
- U$137, U$413: device output:#0X47#0 -> output:#INT#0
- U$138, U$437: device output:PWR0 -> output:#INT#0
- U$139, U$415: device output:PRESSURE0 -> output:#3V3#0
- U$140, U$439: device output:SENSOR0 -> output:#3V3#0
- U$141, U$417: device output:BMP5810 -> output:##CSB##0
- U$142, U$166, U$441, U$442: device output:#GND#0 -> output:##CSB##0
- U$143, U$418: device output:#GND#0 -> output:#ADR#0
- U$144, U$444: device output:#SDI#SDA#0 -> output:#LED#0
- U$145, U$420: device output:#SDI#SDA#0 -> output:#I2C#0
- U$146, U$446: device output:#SCK#SCL#0 -> output:#0X46#0
- U$147, U$422: device output:#SCK#SCL#0 -> output:#0X47#0
- U$148, U$448: device output:#SDO#ADR#0 -> output:PWR0
- U$149, U$424: device output:#SDO#ADR#0 -> output:##CSB##1
- U$151, U$426: device output:#INT#0 -> output:PRESSURE0
- U$152, U$452: device output:#3V3#0 -> output:SENSOR0
- U$153, U$175, U$428, U$475: device output:#3V3#0 -> output:BMP5810
- U$154, U$155, U$430, U$454: device output:##CSB##0 -> output:#GND#0
- U$156, U$432: device output:#ADR#0 -> output:#SDI#SDA#0
- U$157, U$456: device output:#LED#0 -> output:#SDI#SDA#0
- U$158, U$434: device output:#I2C#0 -> output:#SCK#SCL#0
- U$159, U$458: device output:#0X46#0 -> output:#SCK#SCL#0
- U$160, U$436: device output:#0X47#0 -> output:#SDO#ADR#0
- U$161, U$460: device output:PWR0 -> output:#SDO#ADR#0
- U$162, U$438: device output:PRESSURE0 -> output:#INT#0
- U$163, U$462: device output:SENSOR0 -> output:#INT#0
- U$164, U$440: device output:BMP5810 -> output:#3V3#0
- U$165, U$189, U$464, U$465: device output:#GND#0 -> output:#3V3#0
- U$167, U$191, U$466, U$467: device output:#SDI#SDA#0 -> output:##CSB##0
- U$168, U$443: device output:#SDI#SDA#0 -> output:#ADR#0
- U$169, U$469: device output:#SCK#SCL#0 -> output:#LED#0
- U$170, U$445: device output:#SCK#SCL#0 -> output:#I2C#0
- U$171, U$471: device output:#SDO#ADR#0 -> output:#0X46#0
- U$172, U$447: device output:#SDO#ADR#0 -> output:#0X47#0
- U$173, U$473: device output:#INT#0 -> output:PWR0
- U$174, U$449: device output:#INT#0 -> output:##CSB##1
- U$176, U$451: device output:#3V3#0 -> output:PRESSURE0
- U$177, U$477: device output:##CSB##0 -> output:SENSOR0
- U$178, U$200, U$453, U$500: device output:##CSB##0 -> output:BMP5810
- U$179, U$455: device output:#ADR#0 -> output:#GND#0
- U$18: device output:PRESSURE0 -> output:##CSB##1
- U$180, U$479: device output:#LED#0 -> output:#GND#0
- U$181, U$457: device output:#I2C#0 -> output:#SDI#SDA#0
- U$182, U$481: device output:#0X46#0 -> output:#SDI#SDA#0
- U$183, U$459: device output:#0X47#0 -> output:#SCK#SCL#0
- U$184, U$483: device output:PWR0 -> output:#SCK#SCL#0
- U$185, U$461: device output:PRESSURE0 -> output:#SDO#ADR#0
- U$186, U$485: device output:SENSOR0 -> output:#SDO#ADR#0
- U$187, U$463: device output:BMP5810 -> output:#INT#0
- U$188, U$212, U$487, U$488: device output:#GND#0 -> output:#INT#0
- U$190, U$214, U$489, U$490: device output:#SDI#SDA#0 -> output:#3V3#0
- U$192, U$216, U$491, U$492: device output:#SCK#SCL#0 -> output:##CSB##0
- U$193, U$468: device output:#SCK#SCL#0 -> output:#ADR#0
- U$194, U$494: device output:#SDO#ADR#0 -> output:#LED#0
- U$195, U$470: device output:#SDO#ADR#0 -> output:#I2C#0
- U$196, U$496: device output:#INT#0 -> output:#0X46#0
- U$197, U$472: device output:#INT#0 -> output:#0X47#0
- U$198, U$498: device output:#3V3#0 -> output:PWR0
- U$199, U$474: device output:#3V3#0 -> output:##CSB##1
- U$201, U$476: device output:##CSB##0 -> output:PRESSURE0
- U$202: device output:#ADR#0 -> output:SENSOR0
- U$203, U$525: device output:#LED#0 -> output:BMP5810
- U$204, U$480: device output:#I2C#0 -> output:#GND#0
- U$205, U$504: device output:#0X46#0 -> output:#GND#0
- U$206, U$482: device output:#0X47#0 -> output:#SDI#SDA#0
- U$207, U$506: device output:PWR0 -> output:#SDI#SDA#0
- U$208, U$484: device output:PRESSURE0 -> output:#SCK#SCL#0
- U$209, U$508: device output:SENSOR0 -> output:#SCK#SCL#0
- U$210, U$486: device output:BMP5810 -> output:#SDO#ADR#0
- U$211, U$235, U$510, U$511: device output:#GND#0 -> output:#SDO#ADR#0
- U$213, U$237, U$512, U$513: device output:#SDI#SDA#0 -> output:#INT#0
- U$215, U$239, U$514, U$515: device output:#SCK#SCL#0 -> output:#3V3#0
- U$217, U$241, U$516, U$517: device output:#SDO#ADR#0 -> output:##CSB##0
- U$218, U$493: device output:#SDO#ADR#0 -> output:#ADR#0
- U$219, U$519: device output:#INT#0 -> output:#LED#0
- U$22, U$278: device output:SENSOR0 -> output:BMP5810
- U$220, U$495: device output:#INT#0 -> output:#I2C#0
- U$221, U$521: device output:#3V3#0 -> output:#0X46#0
- U$222, U$497: device output:#3V3#0 -> output:#0X47#0
- U$223, U$523: device output:##CSB##0 -> output:PWR0
- U$224, U$499: device output:##CSB##0 -> output:##CSB##1
- U$225, U$478: device output:#ADR#0 -> output:BMP5810
- U$226: device output:#LED#0 -> output:PRESSURE0
- U$227: device output:#I2C#0 -> output:SENSOR0
- U$228, U$550: device output:#0X46#0 -> output:BMP5810
- U$229, U$505: device output:#0X47#0 -> output:#GND#0
- U$23: device output:BMP5810 -> output:PRESSURE0
- U$230, U$529: device output:PWR0 -> output:#GND#0
- U$231, U$507: device output:PRESSURE0 -> output:#SDI#SDA#0
- U$232, U$531: device output:SENSOR0 -> output:#SDI#SDA#0
- U$233, U$509: device output:BMP5810 -> output:#SCK#SCL#0
- U$234, U$258, U$533, U$534: device output:#GND#0 -> output:#SCK#SCL#0
- U$236, U$260, U$535, U$536: device output:#SDI#SDA#0 -> output:#SDO#ADR#0
- U$238, U$262, U$537, U$538: device output:#SCK#SCL#0 -> output:#INT#0
- U$24, U$327: device output:#GND#0 -> output:SENSOR0
- U$240, U$264, U$539, U$540: device output:#SDO#ADR#0 -> output:#3V3#0
- U$242, U$266, U$541, U$542: device output:#INT#0 -> output:##CSB##0
- U$243, U$518: device output:#INT#0 -> output:#ADR#0
- U$244, U$544: device output:#3V3#0 -> output:#LED#0
- U$245, U$520: device output:#3V3#0 -> output:#I2C#0
- U$246, U$546: device output:##CSB##0 -> output:#0X46#0
- U$247, U$522: device output:##CSB##0 -> output:#0X47#0
- U$248: device output:#ADR#0 -> output:PWR0
- U$249: device output:#LED#0 -> output:##CSB##1
- U$250, U$503: device output:#I2C#0 -> output:BMP5810
- U$251: device output:#0X46#0 -> output:PRESSURE0
- U$252: device output:#0X47#0 -> output:SENSOR0
- U$253: device output:PWR0 -> output:BMP5810
- U$254, U$530: device output:PRESSURE0 -> output:#GND#0
- U$255: device output:SENSOR0 -> output:#GND#0
- U$256, U$532: device output:BMP5810 -> output:#SDI#SDA#0
- U$257, U$281: device output:#GND#0 -> output:#SDI#SDA#0
- U$259, U$283: device output:#SDI#SDA#0 -> output:#SCK#SCL#0
- U$261, U$285: device output:#SCK#SCL#0 -> output:#SDO#ADR#0
- U$263, U$287: device output:#SDO#ADR#0 -> output:#INT#0
- U$265, U$289: device output:#INT#0 -> output:#3V3#0
- U$267, U$291: device output:#3V3#0 -> output:##CSB##0
- U$268, U$543: device output:#3V3#0 -> output:#ADR#0
- U$269: device output:##CSB##0 -> output:#LED#0
- U$27, U$303, U$350, U$50: device output:#GND#0 -> output:BMP5810
- U$270, U$545: device output:##CSB##0 -> output:#I2C#0
- U$271: device output:#ADR#0 -> output:#0X46#0
- U$272: device output:#LED#0 -> output:#0X47#0
- U$273: device output:#I2C#0 -> output:PWR0
- U$274: device output:#0X46#0 -> output:##CSB##1
- U$275, U$528: device output:#0X47#0 -> output:BMP5810
- U$276: device output:PWR0 -> output:PRESSURE0
- U$277: device output:PRESSURE0 -> output:SENSOR0
- U$279: device output:BMP5810 -> output:#GND#0
- U$29, U$30, U$305, U$329: device output:#SDI#SDA#0 -> output:#GND#0
- U$293: device output:##CSB##0 -> output:#ADR#0
- U$294: device output:#ADR#0 -> output:#LED#0
- U$295: device output:#LED#0 -> output:#I2C#0
- U$296: device output:#I2C#0 -> output:#0X46#0
- U$297: device output:#0X46#0 -> output:#0X47#0
- U$298: device output:#0X47#0 -> output:PWR0
- U$299: device output:PWR0 -> output:##CSB##1
- U$300: device output:PRESSURE0 -> output:BMP5810
- U$301: device output:SENSOR0 -> output:PRESSURE0
- U$302: device output:BMP5810 -> output:SENSOR0
- U$307, U$31, U$32, U$331: device output:#SCK#SCL#0 -> output:#SDI#SDA#0
- U$309, U$33, U$333, U$34: device output:#SDO#ADR#0 -> output:#SCK#SCL#0
- U$311, U$335, U$35, U$36: device output:#INT#0 -> output:#SDO#ADR#0
- U$313, U$337, U$37, U$38: device output:#3V3#0 -> output:#INT#0
- U$315, U$339, U$39, U$40: device output:##CSB##0 -> output:#3V3#0
- U$317, U$41: device output:#ADR#0 -> output:##CSB##0
- U$318: device output:#LED#0 -> output:#ADR#0
- U$319: device output:#I2C#0 -> output:#LED#0
- U$320: device output:#0X46#0 -> output:#I2C#0
- U$321: device output:#0X47#0 -> output:#0X46#0
- U$322: device output:PWR0 -> output:#0X47#0
- U$323: device output:PRESSURE0 -> output:PWR0
- U$324: device output:SENSOR0 -> output:##CSB##1
- U$326, U$51: device output:#GND#0 -> output:PRESSURE0
- U$328, U$375, U$53, U$75: device output:#SDI#SDA#0 -> output:BMP5810
- U$330, U$354, U$54, U$55: device output:#SCK#SCL#0 -> output:#GND#0
- U$332, U$356, U$56, U$57: device output:#SDO#ADR#0 -> output:#SDI#SDA#0
- U$334, U$358, U$58, U$59: device output:#INT#0 -> output:#SCK#SCL#0
- U$336, U$360, U$60, U$61: device output:#3V3#0 -> output:#SDO#ADR#0
- U$338, U$362, U$62, U$63: device output:##CSB##0 -> output:#INT#0
- U$340, U$64: device output:#ADR#0 -> output:#3V3#0
- U$341, U$42: device output:#LED#0 -> output:##CSB##0
- U$342, U$66: device output:#I2C#0 -> output:##CSB##0
- U$343: device output:#0X46#0 -> output:#ADR#0
- U$344: device output:#0X47#0 -> output:#LED#0
- U$345: device output:PWR0 -> output:#I2C#0
- U$346: device output:PRESSURE0 -> output:#0X46#0
- U$347: device output:SENSOR0 -> output:#0X47#0
- U$348: device output:BMP5810 -> output:PWR0
- U$349, U$74: device output:#GND#0 -> output:##CSB##1
- U$351, U$76: device output:#SDI#SDA#0 -> output:PRESSURE0
- U$352, U$52: device output:#SDI#SDA#0 -> output:SENSOR0
- U$355, U$379, U$79, U$80: device output:#SDO#ADR#0 -> output:#GND#0
- U$357, U$381, U$81, U$82: device output:#INT#0 -> output:#SDI#SDA#0
- U$359, U$383, U$83, U$84: device output:#3V3#0 -> output:#SCK#SCL#0
- U$361, U$385, U$85, U$86: device output:##CSB##0 -> output:#SDO#ADR#0
- U$363, U$87: device output:#ADR#0 -> output:#INT#0
- U$364, U$65: device output:#LED#0 -> output:#3V3#0
- U$365, U$89: device output:#I2C#0 -> output:#3V3#0
- U$366, U$67: device output:#0X46#0 -> output:##CSB##0
- U$367, U$91: device output:#0X47#0 -> output:##CSB##0
- U$368: device output:PWR0 -> output:#ADR#0
- U$369: device output:PRESSURE0 -> output:#LED#0
- U$370: device output:SENSOR0 -> output:#I2C#0
- U$371: device output:BMP5810 -> output:#0X46#0
- U$372, U$97: device output:#GND#0 -> output:#0X47#0
- U$373, U$73: device output:#GND#0 -> output:PWR0
- U$374, U$99: device output:#SDI#SDA#0 -> output:##CSB##1
- U$377, U$77: device output:#SCK#SCL#0 -> output:SENSOR0
- U$387, U$88: device output:#LED#0 -> output:#INT#0
- U$389, U$90: device output:#0X46#0 -> output:#3V3#0
- U$391, U$92: device output:PWR0 -> output:##CSB##0
- U$393: device output:SENSOR0 -> output:#ADR#0
- U$394: device output:BMP5810 -> output:#LED#0
- U$396, U$96: device output:#GND#0 -> output:#0X46#0
- U$398, U$98: device output:#SDI#SDA#0 -> output:PWR0
- U$43: device output:#I2C#0 -> output:#ADR#0
- U$44: device output:#0X46#0 -> output:#LED#0
- U$45: device output:#0X47#0 -> output:#I2C#0
- U$46: device output:PWR0 -> output:#0X46#0
- U$47: device output:PRESSURE0 -> output:#0X47#0
- U$48: device output:SENSOR0 -> output:PWR0
- U$49: device output:BMP5810 -> output:##CSB##1
- U$501: device output:#ADR#0 -> output:PRESSURE0
- U$502: device output:#LED#0 -> output:SENSOR0
- U$524: device output:#ADR#0 -> output:##CSB##1
- U$526: device output:#I2C#0 -> output:PRESSURE0
- U$527: device output:#0X46#0 -> output:SENSOR0
- U$547: device output:#ADR#0 -> output:#0X47#0
- U$548: device output:#LED#0 -> output:PWR0
- U$549: device output:#I2C#0 -> output:##CSB##1
- U$551: device output:#0X47#0 -> output:PRESSURE0
- U$552: device output:PWR0 -> output:SENSOR0
- U$68: device output:#0X47#0 -> output:#ADR#0
- U$69: device output:PWR0 -> output:#LED#0
- U$70: device output:PRESSURE0 -> output:#I2C#0
- U$71: device output:SENSOR0 -> output:#0X46#0
- U$72: device output:BMP5810 -> output:#0X47#0
- U$93: device output:PRESSURE0 -> output:#ADR#0
- U$94: device output:SENSOR0 -> output:#LED#0
- U$95: device output:BMP5810 -> output:#I2C#0
- moved U$142 144.6 mm to (147.3, 1.78), flipped to the bottom
- moved U$298 142.7 mm to (152.4, 46.2), flipped to the top
- moved U$291 142.1 mm to (147.3, 27.7), flipped to the top
- moved U$141 141.8 mm to (147.3, 1.78), turned to 90 degrees
- moved U$144 141.0 mm to (150.5, 13.6), flipped to the bottom, turned to 0 degrees
- moved U$294 141.0 mm to (150.5, 39.5)
- moved U$436 139.3 mm to (144.8, 53.6), turned to 90 degrees
- moved U$143 137.5 mm to (142.2, 17.5), turned to 0 degrees
- moved U$148 137.4 mm to (152.4, 20.3), turned to 0 degrees
- moved U$287 137.1 mm to (149.9, 27.7), flipped to the top
- moved U$281 137.1 mm to (139.7, 27.7), flipped to the top
- moved U$435 136.7 mm to (144.8, 53.6), flipped to the top, turned to 90 degrees
- moved U$149 135.8 mm to (149.5, 7.11), turned to 0 degrees
- moved U$428 134.8 mm to (142.2, 72.1), turned to 0 degrees
- moved U$434 134.6 mm to (142.2, 53.6), turned to 90 degrees
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Connections:
- new net N$145: D21.A, JP83.1
- new net N$146: D21.C, R125.2
- new net N$147: JP84.2, R126.1
- new net N$148: JP85.3, R129.1
- new net N$149: JP85.1, R130.2
- new net N$150: JP86.1, R128.1
- new net N$151: JP86.3, R127.2
- new net N$152: D22.A, JP87.1
- new net N$153: D22.C, R131.2
- new net N$154: JP88.2, R132.1
- new net N$155: JP89.3, R135.1
- new net N$156: JP89.1, R136.2
- new net N$157: JP90.1, R134.1
- new net N$158: JP90.3, R133.2
- new net N$159: D23.A, JP91.1
- new net N$160: D23.C, R137.2
- new net N$161: JP92.2, R138.1
- new net N$162: JP93.3, R141.1
- new net N$163: JP93.1, R142.2
- new net N$164: JP94.1, R140.1
- new net N$165: JP94.3, R139.2
- new net N$166: D24.A, JP95.1
- new net N$167: D24.C, R143.2
- new net N$168: JP96.2, R144.1
- net !CSB!: now also JP4.1
- net !CSB!1: now also JP8.1
- net !CSB!10: now also JP44.1
- net !CSB!11: now also JP48.1
- net !CSB!12: now also JP52.1
- net !CSB!13: now also JP56.1
- net !CSB!14: now also JP60.1
- net !CSB!15: now also JP64.1
- net !CSB!16: now also JP68.1
- net !CSB!17: now also JP72.1
- net !CSB!18: now also JP76.1
- net !CSB!19: now also JP80.1
- net !CSB!2: now also JP12.1
- net !CSB!20: now also JP84.1
- net !CSB!21: now also JP88.1
- net !CSB!22: now also JP92.1
- net !CSB!23: now also JP96.1
- net !CSB!3: now also JP16.1
- net !CSB!4: now also JP20.1
- net !CSB!5: now also JP24.1
- net !CSB!6: now also JP28.1
- net !CSB!7: now also JP32.1
- net !CSB!8: now also JP36.1
- net !CSB!9: now also JP40.1
- net GND1: now also R11.1; no longer R9.1
- net GND10: now also R64.1, R65.1; no longer R54.1, R55.1
- net GND11: now also R70.1, R71.1; no longer R59.1, R60.1
- net GND12: now also R76.1, R77.1; no longer R64.1, R65.1
- net GND13: now also R82.1, R83.1; no longer R69.1, R70.1
- net GND14: now also R88.1, R89.1; no longer R74.1, R75.1
- net GND15: now also R94.1, R95.1; no longer R79.1, R80.1
- net GND16: now also R100.1, R101.1; no longer R84.1, R85.1
- net GND17: now also R106.1, R107.1; no longer R89.1, R90.1
- net GND18: now also R112.1, R113.1; no longer R94.1, R95.1
- net GND19: now also R118.1, R119.1; no longer R100.1, R99.1
- net GND2: now also R16.1, R17.1; no longer R14.1, R15.1
- net GND20: now also R124.1, R125.1; no longer R104.1, R105.1
- net GND21: now also R130.1, R131.1; no longer R109.1, R110.1
- net GND22: now also R136.1, R137.1; no longer R114.1, R115.1
- net GND23: now also R142.1, R143.1; no longer R119.1, R120.1
- net GND3: now also R22.1, R23.1; no longer R19.1, R20.1
- net GND4: now also R28.1, R29.1; no longer R24.1, R25.1
- net GND5: now also R34.1, R35.1; no longer R29.1, R30.1
- net GND6: now also R40.1, R41.1; no longer R34.1, R35.1
- net GND7: now also R46.1, R47.1; no longer R39.1, R40.1
- net GND8: now also R52.1, R53.1; no longer R44.1, R45.1
- net GND9: now also R58.1, R59.1; no longer R49.1, R50.1
- net N$10: now also JP6.1, R8.1; no longer JP5.3, R6.2
- net N$100: now also JP57.1, R88.2; no longer JP50.3, R81.2
- net N$101: now also JP58.1, R86.1; no longer D17.A, JP51.1
- net N$102: now also JP58.3; no longer D17.C
- net N$103: now also D15.A, JP59.1; no longer JP52.3, R88.1
- net N$104: now also D15.C; no longer JP52.1
- net N$105: now also JP60.2, R90.1; no longer JP53.1, R87.1
- net N$106: now also JP61.3, R93.1; no longer JP53.3, R86.2
- net N$107: now also JP61.1, R94.2; no longer D18.A, JP54.1
- net N$108: now also JP62.1, R92.1; no longer D18.C, R90.2
- net N$109: now also JP62.3, R91.2; no longer JP55.3, R93.1
- net N$11: now also JP6.3, R7.2; no longer D2.A, JP6.1
- net N$110: now also D16.A, JP63.1; no longer JP55.1, R94.2
- net N$111: now also D16.C, R95.2; no longer JP56.1, R92.1
- net N$112: now also JP64.2, R96.1; no longer JP56.3, R91.2
- net N$113: now also JP65.3, R99.1; no longer D19.A, JP57.1
- net N$114: now also JP65.1, R100.2; no longer D19.C, R95.2
- net N$115: now also JP66.1; no longer JP58.3
- net N$116: now also JP66.3, R97.2; no longer JP58.1, R99.2
- net N$117: now also D17.A, JP67.1; no longer JP59.1, R97.1
- net N$118: now also D17.C, R101.2; no longer JP59.3, R96.2
- net N$119: now also JP68.2, R102.1; no longer D20.A, JP60.1
- net N$12: now also D2.A, JP7.1; no longer D2.C, R10.2
- net N$120: now also JP69.3, R105.1; no longer D20.C, R100.2
- net N$121: now also JP69.1, R106.2; no longer JP61.3, R103.1
- net N$122: now also JP70.1, R104.1; no longer JP61.1, R104.2
- net N$123: now also JP70.3, R103.2; no longer JP62.1, R102.1
- net N$124: now also D18.A, JP71.1; no longer JP62.3, R101.2
- net N$125: now also D18.C, R107.2; no longer D21.A, JP63.1
- net N$126: now also JP72.2, R108.1; no longer D21.C, R105.2
- net N$127: now also JP73.3, R111.1; no longer JP64.3, R108.1
- net N$128: now also JP73.1, R112.2; no longer JP64.1, R109.2
- net N$129: now also JP74.1, R110.1; no longer JP65.1, R107.1
- net N$13: now also D2.C, R11.2; no longer JP7.3, R13.1
- net N$130: now also JP74.3, R109.2; no longer JP65.3, R106.2
- net N$131: now also D19.A, JP75.1; no longer D22.A, JP66.1
- net N$132: now also D19.C, R113.2; no longer D22.C, R110.2
- net N$133: now also JP76.2, R114.1; no longer JP67.3, R113.1
- net N$134: now also JP77.3, R117.1; no longer JP67.1, R114.2
- net N$135: now also JP77.1, R118.2; no longer JP68.1, R112.1
- net N$136: now also JP78.1, R116.1; no longer JP68.3, R111.2
- net N$137: now also JP78.3, R115.2; no longer D23.A, JP69.1
- net N$138: now also D20.A, JP79.1; no longer D23.C, R115.2
- net N$139: now also D20.C, R119.2; no longer JP70.3, R118.1
- net N$14: now also JP8.2, R12.1; no longer JP7.1, R14.2
- net N$140: now also JP80.2, R120.1; no longer JP70.1, R119.2
- net N$141: now also JP81.3, R123.1; no longer JP71.1, R117.1
- net N$142: now also JP81.1, R124.2; no longer JP71.3, R116.2
- net N$143: now also JP82.1, R122.1; no longer D24.A, JP72.1
- net N$144: now also JP82.3, R121.2; no longer D24.C, R120.2
- net N$15: now also JP9.3, R15.1; no longer JP8.1, R12.1
- net N$16: now also JP9.1, R16.2; no longer JP8.3, R11.2
- net N$17: now also JP10.1, R14.1; no longer D3.A, JP9.1
- net N$18: now also JP10.3, R13.2; no longer D3.C, R15.2
- net N$19: now also D3.A, JP11.1; no longer JP10.3, R18.1
- net N$20: now also D3.C, R17.2; no longer JP10.1, R19.2
- net N$21: now also JP12.2, R18.1; no longer JP11.1, R17.1
- net N$22: now also JP13.3, R21.1; no longer JP11.3, R16.2
- net N$23: now also JP13.1, R22.2; no longer D4.A, JP12.1
- net N$24: now also JP14.1, R20.1; no longer D4.C, R20.2
- net N$25: now also JP14.3, R19.2; no longer JP13.3, R23.1
- net N$26: now also D4.A, JP15.1; no longer JP13.1, R24.2
- net N$27: now also D4.C, R23.2; no longer JP14.1, R22.1
- net N$28: now also JP16.2, R24.1; no longer JP14.3, R21.2
- net N$29: now also JP17.3, R27.1; no longer D5.A, JP15.1
- net N$30: now also JP17.1, R28.2; no longer D5.C, R25.2
- net N$31: now also JP18.1, R26.1; no longer JP16.3, R28.1
- net N$32: now also JP18.3, R25.2; no longer JP16.1, R29.2
- net N$33: now also D5.A, JP19.1; no longer JP17.1, R27.1
- net N$34: now also D5.C, R29.2; no longer JP17.3, R26.2
- net N$35: now also JP20.2, R30.1; no longer D6.A, JP18.1
- net N$36: now also JP21.3, R33.1; no longer D6.C, R30.2
- net N$37: now also JP21.1, R34.2; no longer JP19.3, R33.1
- net N$38: now also JP22.1, R32.1; no longer JP19.1, R34.2
- net N$39: now also JP22.3, R31.2; no longer JP20.1, R32.1
- net N$40: now also D6.A, JP23.1; no longer JP20.3, R31.2
- net N$41: now also D6.C, R35.2; no longer D7.A, JP21.1
- net N$42: now also JP24.2, R36.1; no longer D7.C, R35.2
- net N$43: now also JP25.3, R39.1; no longer JP22.3, R38.1
- net N$44: now also JP25.1, R40.2; no longer JP22.1, R39.2
- net N$45: now also JP26.1, R38.1; no longer JP23.1, R37.1
- net N$46: now also JP26.3, R37.2; no longer JP23.3, R36.2
- net N$47: now also D7.A, JP27.1; no longer D8.A, JP24.1
- net N$48: now also D7.C, R41.2; no longer D8.C, R40.2
- net N$49: now also JP28.2, R42.1; no longer JP25.3, R43.1
- net N$50: now also JP29.3, R45.1; no longer JP25.1, R44.2
- net N$51: now also JP29.1, R46.2; no longer JP26.1, R42.1
- net N$52: now also JP30.1, R44.1; no longer JP26.3, R41.2
- net N$53: now also JP30.3, R43.2; no longer D9.A, JP27.1
- net N$54: now also D8.A, JP31.1; no longer D9.C, R45.2
- net N$55: now also D8.C, R47.2; no longer JP28.3, R48.1
- net N$56: now also JP32.2, R48.1; no longer JP28.1, R49.2
- net N$57: now also JP33.3, R51.1; no longer JP29.1, R47.1
- net N$58: now also JP33.1, R52.2; no longer JP29.3, R46.2
- net N$59: now also JP34.1, R50.1; no longer D10.A, JP30.1
- net N$60: now also JP34.3, R49.2; no longer D10.C, R50.2
- net N$61: now also D9.A, JP35.1; no longer JP31.3, R53.1
- net N$62: now also D9.C, R53.2; no longer JP31.1, R54.2
- net N$63: now also JP36.2, R54.1; no longer JP32.1, R52.1
- net N$64: now also JP37.3, R57.1; no longer JP32.3, R51.2
- net N$65: now also JP37.1, R58.2; no longer D11.A, JP33.1
- net N$66: now also JP38.1, R56.1; no longer D11.C, R55.2
- net N$67: now also JP38.3, R55.2; no longer JP34.3, R58.1
- net N$68: now also D10.A, JP39.1; no longer JP34.1, R59.2
- net N$69: now also D10.C, R59.2; no longer JP35.1, R57.1
- net N$7: now also JP4.2, R6.1; no longer JP4.3, R8.1
- net N$70: now also JP40.2, R60.1; no longer JP35.3, R56.2
- net N$71: now also JP41.3, R63.1; no longer D12.A, JP36.1
- net N$72: now also JP41.1, R64.2; no longer D12.C, R60.2
- net N$73: now also JP42.1, R62.1; no longer JP37.3, R63.1
- net N$74: now also JP42.3, R61.2; no longer JP37.1, R64.2
- net N$75: now also D11.A, JP43.1; no longer JP38.1, R62.1
- net N$76: now also D11.C, R65.2; no longer JP38.3, R61.2
- net N$77: now also JP44.2, R66.1; no longer D13.A, JP39.1
- net N$78: now also JP45.3, R69.1; no longer D13.C, R65.2
- net N$79: now also JP45.1, R70.2; no longer JP40.3, R68.1
- net N$8: now also JP5.3, R9.1; no longer JP4.1, R9.2
- net N$80: now also JP46.1, R68.1; no longer JP40.1, R69.2
- net N$81: now also JP46.3, R67.2; no longer JP41.1, R67.1
- net N$82: now also D12.A, JP47.1; no longer JP41.3, R66.2
- net N$83: now also D12.C, R71.2; no longer D14.A, JP42.1
- net N$84: now also JP48.2, R72.1; no longer D14.C, R70.2
- net N$85: now also JP49.3, R75.1; no longer JP43.3, R73.1
- net N$86: now also JP49.1, R76.2; no longer JP43.1, R74.2
- net N$87: now also JP50.1, R74.1; no longer JP44.1, R72.1
- net N$88: now also JP50.3, R73.2; no longer JP44.3, R71.2
- net N$89: now also D13.A, JP51.1; no longer D15.A, JP45.1
- net N$9: now also R10.2; no longer R7.1
- net N$90: now also D13.C, R77.2; no longer D15.C, R75.2
- net N$91: now also JP52.2; no longer JP46.3
- net N$92: now also JP53.3, R81.1; no longer JP46.1, R79.2
- net N$93: now also JP53.1, R82.2; no longer JP47.1, R77.1
- net N$94: now also JP54.1, R80.1; no longer JP47.3, R76.2
- net N$95: now also JP54.3, R79.2; no longer D16.A, JP48.1
- net N$96: now also D14.A, JP55.1; no longer D16.C, R80.2
- net N$97: now also D14.C, R83.2; no longer JP49.3, R83.1
- net N$98: now also JP56.2, R84.1; no longer JP49.1, R84.2
- net N$99: now also JP57.3, R87.1; no longer JP50.1, R82.1
- net SCK/SCL1: now also R8.2; no longer R7.2
- net SCK/SCL10: now also R62.2; no longer R52.2
- net SCK/SCL11: now also R68.2; no longer R57.2
- net SCK/SCL12: now also R74.2; no longer R62.2
- net SCK/SCL13: now also R80.2; no longer R67.2
- net SCK/SCL14: now also R86.2; no longer R72.2
- net SCK/SCL15: now also R92.2; no longer R77.2
- net SCK/SCL16: now also R98.2; no longer R82.2
- net SCK/SCL17: now also R104.2; no longer R87.2
- net SCK/SCL18: now also R110.2; no longer R92.2
- net SCK/SCL19: now also R116.2; no longer R97.2
- net SCK/SCL2: now also R14.2; no longer R12.2
- net SCK/SCL20: now also R122.2; no longer R102.2
- net SCK/SCL21: now also R128.2; no longer R107.2
- net SCK/SCL22: now also R134.2; no longer R112.2
- net SCK/SCL23: now also R140.2; no longer R117.2
- net SCK/SCL3: now also R20.2; no longer R17.2
- net SCK/SCL4: now also R26.2; no longer R22.2
- net SCK/SCL5: now also R32.2; no longer R27.2
- net SCK/SCL6: now also R38.2; no longer R32.2
- net SCK/SCL7: now also R44.2; no longer R37.2
- net SCK/SCL8: now also R50.2; no longer R42.2
- net SCK/SCL9: now also R56.2; no longer R47.2
- net SDI/SDA1: now also R7.1; no longer R6.1
- net SDI/SDA10: now also R61.1; no longer R51.1
- net SDI/SDA11: now also R67.1; no longer R56.1
- net SDI/SDA12: now also R73.1; no longer R61.1
- net SDI/SDA13: now also R79.1; no longer R66.1
- net SDI/SDA14: now also R85.1; no longer R71.1
- net SDI/SDA15: now also R91.1; no longer R76.1
- net SDI/SDA16: now also R97.1; no longer R81.1
- net SDI/SDA17: now also R103.1; no longer R86.1
- net SDI/SDA18: now also R109.1; no longer R91.1
- net SDI/SDA19: now also R115.1; no longer R96.1
- net SDI/SDA2: now also R13.1; no longer R11.1
- net SDI/SDA20: now also R121.1; no longer R101.1
- net SDI/SDA21: now also R127.1; no longer R106.1
- net SDI/SDA22: now also R133.1; no longer R111.1
- net SDI/SDA23: now also R139.1; no longer R116.1
- net SDI/SDA3: now also R19.1; no longer R16.1
- net SDI/SDA4: now also R25.1; no longer R21.1
- net SDI/SDA5: now also R31.1; no longer R26.1
- net SDI/SDA6: now also R37.1; no longer R31.1
- net SDI/SDA7: now also R43.1; no longer R36.1
- net SDI/SDA8: now also R49.1; no longer R41.1
- net SDI/SDA9: now also R55.1; no longer R46.1
- net SDO/ADR1: now also JP5.2; no longer JP4.2
- net SDO/ADR10: now also JP41.2; no longer JP31.2
- net SDO/ADR11: now also JP45.2; no longer JP34.2
- net SDO/ADR12: now also JP49.2; no longer JP37.2
- net SDO/ADR13: now also JP53.2; no longer JP40.2
- net SDO/ADR14: now also JP57.2; no longer JP43.2
- net SDO/ADR15: now also JP61.2; no longer JP46.2
- net SDO/ADR16: now also JP65.2; no longer JP49.2
- net SDO/ADR17: now also JP69.2; no longer JP52.2
- net SDO/ADR18: now also JP73.2; no longer JP55.2
- net SDO/ADR19: now also JP77.2; no longer JP58.2
- net SDO/ADR2: now also JP9.2; no longer JP7.2
- net SDO/ADR20: now also JP81.2; no longer JP61.2
- net SDO/ADR21: now also JP85.2; no longer JP64.2
- net SDO/ADR22: now also JP89.2; no longer JP67.2
- net SDO/ADR23: now also JP93.2; no longer JP70.2
- net SDO/ADR3: now also JP13.2; no longer JP10.2
- net SDO/ADR4: now also JP17.2; no longer JP13.2
- net SDO/ADR5: now also JP21.2; no longer JP16.2
- net SDO/ADR6: now also JP25.2; no longer JP19.2
- net SDO/ADR7: now also JP29.2; no longer JP22.2
- net SDO/ADR8: now also JP33.2; no longer JP25.2
- net SDO/ADR9: now also JP37.2; no longer JP28.2
- net VDD: now also R6.2
- net VDD1: now also JP7.2, R12.2, R9.2; no longer JP5.2, R8.2
- net VDD10: now also JP42.2, JP43.2, R63.2, R66.2; no longer JP32.2, JP33.2, R53.2
- net VDD11: now also JP46.2, JP47.2, R69.2, R72.2; no longer JP35.2, JP36.2, R58.2
- net VDD12: now also JP50.2, JP51.2, R75.2, R78.2; no longer JP38.2, JP39.2, R63.2
- net VDD13: now also JP54.2, JP55.2, R81.2, R84.2; no longer JP41.2, JP42.2, R68.2
- net VDD14: now also JP58.2, JP59.2, R87.2, R90.2; no longer JP44.2, JP45.2, R73.2
- net VDD15: now also JP62.2, JP63.2, R93.2, R96.2; no longer JP47.2, JP48.2, R78.2
- net VDD16: now also JP66.2, JP67.2, R102.2, R99.2; no longer JP50.2, JP51.2, R83.2
- net VDD17: now also JP70.2, JP71.2, R105.2, R108.2; no longer JP53.2, JP54.2, R88.2
- net VDD18: now also JP74.2, JP75.2, R111.2, R114.2; no longer JP56.2, JP57.2, R93.2
- net VDD19: now also JP78.2, JP79.2, R117.2, R120.2; no longer JP59.2, JP60.2, R98.2
- net VDD2: now also JP10.2, JP11.2, R15.2, R18.2; no longer JP8.2, JP9.2, R13.2
- net VDD20: now also JP82.2, JP83.2, R123.2, R126.2; no longer JP62.2, JP63.2, R103.2
- net VDD21: now also JP86.2, JP87.2, R129.2, R132.2; no longer JP65.2, JP66.2, R108.2
- net VDD22: now also JP90.2, JP91.2, R135.2, R138.2; no longer JP68.2, JP69.2, R113.2
- net VDD23: now also JP94.2, JP95.2, R141.2, R144.2; no longer JP71.2, JP72.2, R118.2
- net VDD3: now also JP14.2, JP15.2, R21.2, R24.2; no longer JP11.2, JP12.2, R18.2
- net VDD4: now also JP18.2, JP19.2, R27.2, R30.2; no longer JP14.2, JP15.2, R23.2
- net VDD5: now also JP22.2, JP23.2, R33.2, R36.2; no longer JP17.2, JP18.2, R28.2
- net VDD6: now also JP26.2, JP27.2, R39.2, R42.2; no longer JP20.2, JP21.2, R33.2
- net VDD7: now also JP30.2, JP31.2, R45.2, R48.2; no longer JP23.2, JP24.2, R38.2
- net VDD8: now also JP34.2, JP35.2, R51.2, R54.2; no longer JP26.2, JP27.2, R43.2
- net VDD9: now also JP38.2, JP39.2, R57.2, R60.2; no longer JP29.2, JP30.2, R48.2
Routing:
- net N$166: track 0.00 -> 5.10 mm, vias 0 -> 1
- net N$159: track 0.00 -> 5.10 mm, vias 0 -> 1
- net N$152: track 0.00 -> 5.10 mm, vias 0 -> 1
- net N$145: track 0.00 -> 5.10 mm, vias 0 -> 1
- net VDD9: track 46.1 -> 50.3 mm
- net VDD7: track 46.1 -> 50.3 mm
- net VDD5: track 46.1 -> 50.3 mm
- net VDD11: track 46.1 -> 50.3 mm
- net VDD10: track 46.1 -> 50.3 mm
- net VDD6: track 46.1 -> 50.3 mm
- net VDD4: track 46.1 -> 50.3 mm
- net VDD3: track 46.1 -> 50.3 mm
- net VDD23: track 46.1 -> 50.3 mm
- net VDD22: track 46.1 -> 50.3 mm
- net VDD21: track 46.1 -> 50.3 mm
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