File: Production/Qwiic Micro/SparkFun_Pressure_Sensor_BMP581_Qwiic_Micro-Panel.brd (EAGLE design)
At the start: 84.6 x 170.2 mm, 2502 parts, among them J1 QWIIC_RIGHT_ANGLE, J10 QWIIC_RIGHT_ANGLE, J100 QWIIC_RIGHT_ANGLE, J103 QWIIC_RIGHT_ANGLE, J106 QWIIC_RIGHT_ANGLE, J109 QWIIC_RIGHT_ANGLE, J112 QWIIC_RIGHT_ANGLE, J115 QWIIC_RIGHT_ANGLE, J118 QWIIC_RIGHT_ANGLE, J121 QWIIC_RIGHT_ANGLE, J124 QWIIC_RIGHT_ANGLE, J127 QWIIC_RIGHT_ANGLE, J13 QWIIC_RIGHT_ANGLE, J130 QWIIC_RIGHT_ANGLE, J133 QWIIC_RIGHT_ANGLE, J136 QWIIC_RIGHT_ANGLE, J139 QWIIC_RIGHT_ANGLE, J142 QWIIC_RIGHT_ANGLE, J145 QWIIC_RIGHT_ANGLE, J148 QWIIC_RIGHT_ANGLE, J151 QWIIC_RIGHT_ANGLE, J154 QWIIC_RIGHT_ANGLE, J157 QWIIC_RIGHT_ANGLE, J16 QWIIC_RIGHT_ANGLE, J160 QWIIC_RIGHT_ANGLE, J163 QWIIC_RIGHT_ANGLE, J166 QWIIC_RIGHT_ANGLE, J169 QWIIC_RIGHT_ANGLE, J172 QWIIC_RIGHT_ANGLE, J175 QWIIC_RIGHT_ANGLE, J178 QWIIC_RIGHT_ANGLE, J181 QWIIC_RIGHT_ANGLE, J184 QWIIC_RIGHT_ANGLE, J187 QWIIC_RIGHT_ANGLE, J19 QWIIC_RIGHT_ANGLE, J190 QWIIC_RIGHT_ANGLE, J22 QWIIC_RIGHT_ANGLE, J25 QWIIC_RIGHT_ANGLE, J28 QWIIC_RIGHT_ANGLE, J31 QWIIC_RIGHT_ANGLE, J34 QWIIC_RIGHT_ANGLE, J37 QWIIC_RIGHT_ANGLE, J4 QWIIC_RIGHT_ANGLE, J40 QWIIC_RIGHT_ANGLE, J43 QWIIC_RIGHT_ANGLE, J46 QWIIC_RIGHT_ANGLE, J49 QWIIC_RIGHT_ANGLE, J52 QWIIC_RIGHT_ANGLE, J55 QWIIC_RIGHT_ANGLE, J58 QWIIC_RIGHT_ANGLE, J61 QWIIC_RIGHT_ANGLE, J64 QWIIC_RIGHT_ANGLE, J67 QWIIC_RIGHT_ANGLE, J7 QWIIC_RIGHT_ANGLE, J70 QWIIC_RIGHT_ANGLE, J73 QWIIC_RIGHT_ANGLE, J76 QWIIC_RIGHT_ANGLE, J79 QWIIC_RIGHT_ANGLE, J82 QWIIC_RIGHT_ANGLE, J85 QWIIC_RIGHT_ANGLE, J88 QWIIC_RIGHT_ANGLE, J91 QWIIC_RIGHT_ANGLE, J94 QWIIC_RIGHT_ANGLE, J97 QWIIC_RIGHT_ANGLE, U1 BMP581, U10 BMP581, U11 BMP581, U12 BMP581, U13 BMP581, U14 BMP581, U15 BMP581, U16 BMP581, U17 BMP581, U18 BMP581, U19 BMP581, U2 BMP581, U20 BMP581, U21 BMP581, U22 BMP581, U23 BMP581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

Commit message: Add production files for reds
Connections:
- net SCK/SCL renamed SCL
- net SCK/SCL1 renamed SCL1
- net SCK/SCL10 renamed SCL10
- net SCK/SCL11 renamed SCL11
- net SCK/SCL12 renamed SCL12
- net SCK/SCL13 renamed SCL13
- net SCK/SCL14 renamed SCL14
- net SCK/SCL15 renamed SCL15
- net SCK/SCL16 renamed SCL16
- net SCK/SCL17 renamed SCL17
- net SCK/SCL18 renamed SCL18
- net SCK/SCL19 renamed SCL19
- net SCK/SCL2 renamed SCL2
- net SCK/SCL20 renamed SCL20
- net SCK/SCL21 renamed SCL21
- net SCK/SCL22 renamed SCL22
- net SCK/SCL23 renamed SCL23
- net SCK/SCL24 renamed SCL24
- net SCK/SCL25 renamed SCL25
- net SCK/SCL26 renamed SCL26
- net SCK/SCL27 renamed SCL27
- net SCK/SCL28 renamed SCL28
- net SCK/SCL29 renamed SCL29
- net SCK/SCL3 renamed SCL3
- net SCK/SCL30 renamed SCL30
- net SCK/SCL31 renamed SCL31
- net SCK/SCL32 renamed SCL32
- net SCK/SCL33 renamed SCL33
- net SCK/SCL34 renamed SCL34
- net SCK/SCL35 renamed SCL35
- net SCK/SCL36 renamed SCL36
- net SCK/SCL37 renamed SCL37
- net SCK/SCL38 renamed SCL38
- net SCK/SCL39 renamed SCL39
- net SCK/SCL4 renamed SCL4
- net SCK/SCL40 renamed SCL40
- net SCK/SCL41 renamed SCL41
- net SCK/SCL42 renamed SCL42
- net SCK/SCL43 renamed SCL43
- net SCK/SCL44 renamed SCL44
- net SCK/SCL45 renamed SCL45
- net SCK/SCL46 renamed SCL46
- net SCK/SCL47 renamed SCL47
- net SCK/SCL48 renamed SCL48
- net SCK/SCL49 renamed SCL49
- net SCK/SCL5 renamed SCL5
- net SCK/SCL50 renamed SCL50
- net SCK/SCL51 renamed SCL51
- net SCK/SCL52 renamed SCL52
- net SCK/SCL53 renamed SCL53
- net SCK/SCL54 renamed SCL54
- net SCK/SCL55 renamed SCL55
- net SCK/SCL56 renamed SCL56
- net SCK/SCL57 renamed SCL57
- net SCK/SCL58 renamed SCL58
- net SCK/SCL59 renamed SCL59
- net SCK/SCL6 renamed SCL6
- net SCK/SCL60 renamed SCL60
- net SCK/SCL61 renamed SCL61
- net SCK/SCL62 renamed SCL62
- net SCK/SCL63 renamed SCL63
- net SCK/SCL7 renamed SCL7
- net SCK/SCL8 renamed SCL8
- net SCK/SCL9 renamed SCL9
- net SDI/SDA renamed SDA
- net SDI/SDA1 renamed SDA1
- net SDI/SDA10 renamed SDA10
- net SDI/SDA11 renamed SDA11
- net SDI/SDA12 renamed SDA12
- net SDI/SDA13 renamed SDA13
- net SDI/SDA14 renamed SDA14
- net SDI/SDA15 renamed SDA15
- net SDI/SDA16 renamed SDA16
- net SDI/SDA17 renamed SDA17
- net SDI/SDA18 renamed SDA18
- net SDI/SDA19 renamed SDA19
- net SDI/SDA2 renamed SDA2
- net SDI/SDA20 renamed SDA20
- net SDI/SDA21 renamed SDA21
- net SDI/SDA22 renamed SDA22
- net SDI/SDA23 renamed SDA23
- net SDI/SDA24 renamed SDA24
- net SDI/SDA25 renamed SDA25
- net SDI/SDA26 renamed SDA26
- net SDI/SDA27 renamed SDA27
- net SDI/SDA28 renamed SDA28
- net SDI/SDA29 renamed SDA29
- net SDI/SDA3 renamed SDA3
- net SDI/SDA30 renamed SDA30
- net SDI/SDA31 renamed SDA31
- net SDI/SDA32 renamed SDA32
- net SDI/SDA33 renamed SDA33
- net SDI/SDA34 renamed SDA34
- net SDI/SDA35 renamed SDA35
- net SDI/SDA36 renamed SDA36
- net SDI/SDA37 renamed SDA37
- net SDI/SDA38 renamed SDA38
- net SDI/SDA39 renamed SDA39
- net SDI/SDA4 renamed SDA4
- net SDI/SDA40 renamed SDA40
- net SDI/SDA41 renamed SDA41
- net SDI/SDA42 renamed SDA42
- net SDI/SDA43 renamed SDA43
- net SDI/SDA44 renamed SDA44
- net SDI/SDA45 renamed SDA45
- net SDI/SDA46 renamed SDA46
- net SDI/SDA47 renamed SDA47
- net SDI/SDA48 renamed SDA48
- net SDI/SDA49 renamed SDA49
- net SDI/SDA5 renamed SDA5
- net SDI/SDA50 renamed SDA50
- net SDI/SDA51 renamed SDA51
- net SDI/SDA52 renamed SDA52
- net SDI/SDA53 renamed SDA53
- net SDI/SDA54 renamed SDA54
- net SDI/SDA55 renamed SDA55
- net SDI/SDA56 renamed SDA56
- net SDI/SDA57 renamed SDA57
- net SDI/SDA58 renamed SDA58
- net SDI/SDA59 renamed SDA59
- net SDI/SDA6 renamed SDA6
- net SDI/SDA60 renamed SDA60
- net SDI/SDA61 renamed SDA61
- net SDI/SDA62 renamed SDA62
- net SDI/SDA63 renamed SDA63
- net SDI/SDA7 renamed SDA7
- net SDI/SDA8 renamed SDA8
- net SDI/SDA9 renamed SDA9
- net SDO/ADR renamed ADR
- net SDO/ADR1 renamed ADR1
- net SDO/ADR10 renamed ADR10
- net SDO/ADR11 renamed ADR11
- net SDO/ADR12 renamed ADR12
- net SDO/ADR13 renamed ADR13
- net SDO/ADR14 renamed ADR14
- net SDO/ADR15 renamed ADR15
- net SDO/ADR16 renamed ADR16
- net SDO/ADR17 renamed ADR17
- net SDO/ADR18 renamed ADR18
- net SDO/ADR19 renamed ADR19
- net SDO/ADR2 renamed ADR2
- net SDO/ADR20 renamed ADR20
- net SDO/ADR21 renamed ADR21
- net SDO/ADR22 renamed ADR22
- net SDO/ADR23 renamed ADR23
- net SDO/ADR24 renamed ADR24
- net SDO/ADR25 renamed ADR25
- net SDO/ADR26 renamed ADR26
- net SDO/ADR27 renamed ADR27
- net SDO/ADR28 renamed ADR28
- net SDO/ADR29 renamed ADR29
- net SDO/ADR3 renamed ADR3
- net SDO/ADR30 renamed ADR30
- net SDO/ADR31 renamed ADR31
- net SDO/ADR32 renamed ADR32
- net SDO/ADR33 renamed ADR33
- net SDO/ADR34 renamed ADR34
- net SDO/ADR35 renamed ADR35
- net SDO/ADR36 renamed ADR36
- net SDO/ADR37 renamed ADR37
- net SDO/ADR38 renamed ADR38
- net SDO/ADR39 renamed ADR39
- net SDO/ADR4 renamed ADR4
- net SDO/ADR40 renamed ADR40
- net SDO/ADR41 renamed ADR41
- net SDO/ADR42 renamed ADR42
- net SDO/ADR43 renamed ADR43
- net SDO/ADR44 renamed ADR44
- net SDO/ADR45 renamed ADR45
- net SDO/ADR46 renamed ADR46
- net SDO/ADR47 renamed ADR47
- net SDO/ADR48 renamed ADR48
- net SDO/ADR49 renamed ADR49
- net SDO/ADR5 renamed ADR5
- net SDO/ADR50 renamed ADR50
- net SDO/ADR51 renamed ADR51
- net SDO/ADR52 renamed ADR52
- net SDO/ADR53 renamed ADR53
- net SDO/ADR54 renamed ADR54
- net SDO/ADR55 renamed ADR55
- net SDO/ADR56 renamed ADR56
- net SDO/ADR57 renamed ADR57
- net SDO/ADR58 renamed ADR58
- net SDO/ADR59 renamed ADR59
- net SDO/ADR6 renamed ADR6
- net SDO/ADR60 renamed ADR60
- net SDO/ADR61 renamed ADR61
- net SDO/ADR62 renamed ADR62
- net SDO/ADR63 renamed ADR63
- net SDO/ADR7 renamed ADR7
- net SDO/ADR8 renamed ADR8
- net SDO/ADR9 renamed ADR9
- removed net !CSB!: U1.6
- removed net !CSB!1: U2.6
- removed net !CSB!10: U11.6
- removed net !CSB!11: U12.6
- removed net !CSB!12: U13.6
- removed net !CSB!13: U14.6
- removed net !CSB!14: U15.6
- removed net !CSB!15: U16.6
- removed net !CSB!16: U17.6
- removed net !CSB!17: U18.6
- removed net !CSB!18: U19.6
- removed net !CSB!19: U20.6
- removed net !CSB!2: U3.6
- removed net !CSB!20: U21.6
- removed net !CSB!21: U22.6
- removed net !CSB!22: U23.6
- removed net !CSB!23: U24.6
- removed net !CSB!24: U25.6
- removed net !CSB!25: U26.6
- removed net !CSB!26: U27.6
- removed net !CSB!27: U28.6
- removed net !CSB!28: U29.6
- removed net !CSB!29: U30.6
- removed net !CSB!3: U4.6
- removed net !CSB!30: U31.6
- removed net !CSB!31: U32.6
- removed net !CSB!32: U33.6
- removed net !CSB!33: U34.6
- removed net !CSB!34: U35.6
- removed net !CSB!35: U36.6
- removed net !CSB!36: U37.6
- removed net !CSB!37: U38.6
- removed net !CSB!38: U39.6
- removed net !CSB!39: U40.6
- removed net !CSB!4: U5.6
- removed net !CSB!40: U41.6
- removed net !CSB!41: U42.6
- removed net !CSB!42: U43.6
- removed net !CSB!43: U44.6
- removed net !CSB!44: U45.6
- removed net !CSB!45: U46.6
- removed net !CSB!46: U47.6
- removed net !CSB!47: U48.6
- removed net !CSB!48: U49.6
- removed net !CSB!49: U50.6
- removed net !CSB!5: U6.6
- removed net !CSB!50: U51.6
- removed net !CSB!51: U52.6
- removed net !CSB!52: U53.6
- removed net !CSB!53: U54.6
- removed net !CSB!54: U55.6
- removed net !CSB!55: U56.6
- removed net !CSB!56: U57.6
- removed net !CSB!57: U58.6
- removed net !CSB!58: U59.6
- removed net !CSB!59: U60.6
- removed net !CSB!6: U7.6
- removed net !CSB!60: U61.6
- removed net !CSB!61: U62.6
- removed net !CSB!62: U63.6
- removed net !CSB!63: U64.6
- removed net !CSB!7: U8.6
- removed net !CSB!8: U9.6
- removed net !CSB!9: U10.6
- net VDD: now also U1.6
- net VDD1: now also U2.6
- net VDD10: now also U11.6
- net VDD11: now also U12.6
- net VDD12: now also U13.6
- net VDD13: now also U14.6
- net VDD14: now also U15.6
- net VDD15: now also U16.6
- net VDD16: now also U17.6
- net VDD17: now also U18.6
- net VDD18: now also U19.6
- net VDD19: now also U20.6
- net VDD2: now also U3.6
- net VDD20: now also U21.6
- net VDD21: now also U22.6
- net VDD22: now also U23.6
- net VDD23: now also U24.6
- net VDD24: now also U25.6
- net VDD25: now also U26.6
- net VDD26: now also U27.6
- net VDD27: now also U28.6
- net VDD28: now also U29.6
- net VDD29: now also U30.6
- net VDD3: now also U4.6
- net VDD30: now also U31.6
- net VDD31: now also U32.6
- net VDD32: now also U33.6
- net VDD33: now also U34.6
- net VDD34: now also U35.6
- net VDD35: now also U36.6
- net VDD36: now also U37.6
- net VDD37: now also U38.6
- net VDD38: now also U39.6
- net VDD39: now also U40.6
- net VDD4: now also U5.6
- net VDD40: now also U41.6
- net VDD41: now also U42.6
- net VDD42: now also U43.6
- net VDD43: now also U44.6
- net VDD44: now also U45.6
- net VDD45: now also U46.6
- net VDD46: now also U47.6
- net VDD47: now also U48.6
- net VDD48: now also U49.6
- net VDD49: now also U50.6
- net VDD5: now also U6.6
- net VDD50: now also U51.6
- net VDD51: now also U52.6
- net VDD52: now also U53.6
- net VDD53: now also U54.6
- net VDD54: now also U55.6
- net VDD55: now also U56.6
- net VDD56: now also U57.6
- net VDD57: now also U58.6
- net VDD58: now also U59.6
- net VDD59: now also U60.6
- net VDD6: now also U7.6
- net VDD60: now also U61.6
- net VDD61: now also U62.6
- net VDD62: now also U63.6
- net VDD63: now also U64.6
- net VDD7: now also U8.6
- net VDD8: now also U9.6
- net VDD9: now also U10.6
Routing:
- net VDD35: track 17.2 -> 18.2 mm, vias 2 -> 3
- net VDD34: track 17.2 -> 18.2 mm, vias 2 -> 3
- net VDD8: track 17.2 -> 18.2 mm, vias 2 -> 3
- net VDD51: track 17.2 -> 18.2 mm, vias 2 -> 3
- net VDD50: track 17.2 -> 18.2 mm, vias 2 -> 3
- net VDD39: track 17.2 -> 18.2 mm, vias 2 -> 3
- net VDD38: track 17.2 -> 18.2 mm, vias 2 -> 3
- net VDD37: track 17.2 -> 18.2 mm, vias 2 -> 3
- net VDD36: track 17.2 -> 18.2 mm, vias 2 -> 3
- net VDD33: track 17.2 -> 18.2 mm, vias 2 -> 3
- net VDD32: track 17.2 -> 18.2 mm, vias 2 -> 3
- net VDD11: track 17.2 -> 18.2 mm, vias 2 -> 3
- net VDD10: track 17.2 -> 18.2 mm, vias 2 -> 3
- net VDD9: track 17.2 -> 18.2 mm, vias 2 -> 3
- net VDD7: track 17.2 -> 18.2 mm, vias 2 -> 3
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